File: hardware/W5500_PA_PTT_Control/kicad/w5500-esp32.kicad_pcb (KiCad board)
At the start: 4 copper layers, 72 x 115 mm, 27 parts, among them J1 ESP32_DevKitC_Socket_40P_25.4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, J2 DC_IN_13V8, J5 Power, J6 PTT_ON, J7 LED_PWR, J8 LED_12V, Q1 2SC1815, Q3 2SC1815, Q5 2SJ334, U1 TA48033S, U2 L7805

Commit message: W5500制御基板: Shonan_Lite-RasPI5版の最新(基板Rev.1.1・仕様書Rev.2.7)に合わせる
KiCadデータ(放熱器の取付ピン穴・3Dモデル)、JLCPCB発注データ、実装図・3D画像、
ケース(RJ45角穴の実測修正・蓋の文字)、接続一覧をPi5版からコピー。
仕様書は連携部分を残し、Rev.2.7の変更だけを反映してWord/PDFを作り直した。

Co-Authored-By: Claude Opus 5.5 <noreply@anthropic.com>
Parts:
- added HS1: 105054, project_footprints:Heatsink_GEC_20PB020_Pins_P12.5mm, F.Cu at (118.7, 75.0)
- added HS2: 105054, project_footprints:Heatsink_GEC_20PB020_Pins_P12.5mm, F.Cu at (118.7, 97.0)
- added HS3: 105054, project_footprints:Heatsink_GEC_20PB020_Pins_P12.5mm, F.Cu at (118.7, 119.0)
Routing:
- net /PTT_ON: track 66.9 -> 68.7 mm
Other:
- board text added: "W5500 PA/PTT Control Rev.1.1"
- board text added: "放熱器 Q5 20x20 (M3穴 高さ19)"
- board text added: "放熱器 U1 20x20 (M3穴 高さ19)"
- board text added: "放熱器 U2 20x20 (M3穴 高さ19)"
- board text removed: "W5500 PA/PTT Control Rev.1.0"
- board text removed: "放熱器 Q5 20x20 (M3穴 高さ18)"
- board text removed: "放熱器 U1 20x20 (M3穴 高さ18)"
- board text removed: "放熱器 U2 20x20 (M3穴 高さ18)"
